File: PCB/Starbie.kicad_pcb (KiCad board)
At the start: 2 copper layers, 50 x 75 mm, 8 parts, among them J1 Conn_01x04_Pin, J2 Conn_01x08_Pin, SW1 SW_Push, SW2 SW_Push, U1 XIAO-ESP32-C3-SMD, U2 DHT11

Commit message: did the actual pcb. added new silkscreens, on off switch, and finalized corner as well as getting all the firmware done
Parts:
- added G***: LOGO, KicadMods:FroggyFace, F.Cu at (186.5, 104.0)
- added G***: LOGO, KicadMods:EnaMural, B.Cu at (169.0, 80.0)
- added G***: LOGO, KicadMods:EnaEye, B.Cu at (154.0, 39.0)
- added R2: 10k, Resistor_THT:R_Axial_DIN0204_L3.6mm_D1.6mm_P7.62mm_Horizontal, F.Cu at (170.5, 102.2)
- added SW3: SW_SPDT, Connector_PinHeader_2.54mm:PinHeader_1x03_P2.54mm_Horizontal, F.Cu at (171.3, 93.3)
Connections:
- U1 pad 7: unconnected-(U1-D6-Pad7) -> /GPIO6
Routing:
- net GND: track 0.00 -> 297.2 mm
- net +3.3V: track 0.00 -> 138.3 mm
- net /SDA: track 0.00 -> 102.8 mm, vias 0 -> 3
- net /SCL: track 0.00 -> 73.0 mm, vias 0 -> 1
- net /DHT11 DATA: track 0.00 -> 49.2 mm
- net /GPIO2: track 0.00 -> 41.4 mm, vias 0 -> 2
- net /GPIO3: track 0.00 -> 32.9 mm, vias 0 -> 1
- net /GPIO6: track 0.00 -> 26.1 mm, vias 0 -> 2
- net Net-(SW3-C): track 0.00 -> 4.21 mm
