File: PCB/Starbie.kicad_sch (KiCad schematic)
At the start: 7 parts, among them J1 Conn_01x04_Pin, J2 Conn_01x08_Pin, SW1 SW_Push, SW2 SW_Push, U1 XIAO-ESP32-C3-SMD, U2 DHT11

Commit message: did the actual pcb. added new silkscreens, on off switch, and finalized corner as well as getting all the firmware done
Parts:
- added R2: 10k, Resistor_THT:R_Axial_DIN0204_L3.6mm_D1.6mm_P7.62mm_Horizontal, symbol Device:R
- added SW3: SW_SPDT, Connector_PinHeader_2.54mm:PinHeader_1x03_P2.54mm_Horizontal, symbol Switch:SW_SPDT
Connections:
- net +3.3V: now also R2.2
- net GND: now also SW3.1 (A)
- net GPIO6: now reaches U1.7 (D6)
- net GPIO6: now also SW3.2 (B)
- new net: R2.1, SW3.3 (C)
- no-connect marks 17 -> 16
